Commit message: Updated Camera Position

File: turtlebot3_description/urdf/turtlebot3_burger.urdf.xacro (robot description, xacro)
@@ -140,3 +140,16 @@
     </inertial>
   </link>
+  <joint name="camera_joint" type="fixed">
+     <parent link="base_link"/>
+     <child link="camera_link"/>
+     <origin rpy="1.396263441 3.141592 1.57079633" xyz="0.042 0 0.105"/>
+    </joint>
+  <link name="camera_link">
+    <visual>
+      <geometry>
+        <cylinder length="0.015" radius="0.0075"/>
+      </geometry>
+      <material name="grey"/>
+    </visual>
+  </link>
 </robot>

Commit message: Rotated LIDAR by 180° to make room for intel RealSense camera

File: turtlebot3_description/urdf/turtlebot3_burger.urdf.xacro (robot description, xacro)
@@ -116,5 +116,5 @@
     <parent link="base_link"/>
     <child link="base_scan"/>
-    <origin xyz="-0.032 0 0.172" rpy="0 0 0"/>
+    <origin xyz="-0.032 0 0.172" rpy="0 0 3.141592"/>
   </joint>
   <link name="base_scan">

Commit message: Added RealSense joint

File: turtlebot3_description/urdf/turtlebot3_burger.urdf.xacro (robot description, xacro)
@@ -153,3 +153,16 @@
     </visual>
   </link>
+  <joint name="realsense_joint" type="fixed">
+     <parent link="base_link"/>
+     <child link="realsense_link"/>
+     <origin rpy="0 0 0" xyz="0.042 0 0.15"/>
+    </joint>
+  <link name="realsense_link">
+    <visual>
+      <geometry>
+        <cylinder length="0.015" radius="0.0075"/>
+      </geometry>
+      <material name="grey"/>
+    </visual>
+  </link>
 </robot>
